File: mc68681-duart/mc68681-duart-basic/design/kicad/mc68681-basic/mc68681-basic.sch (KiCad schematic (older format))
At the start: 30 parts, among them IC1 XR68C681CJTR-F, IC2 74HCT245, IC3 74HCT245, IC4 74HCT245, IC5 74125, IC6 IC6_DECO.PLD, IC7 IC7_UART_.PLD, J1 Conn_02x32_Odd_Even, J2 EXTBUS, J3 UART_A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

Commit message: Fix broken Kicad library
Parts:
- IC1: symbol XR68C681:XR68C681CJTR-F -> mc68681-basic-rescue:XR68C681CJTR-F-XR68C681
Changed lines of the file:
@@
 	2800 5700 3700 5700
 $Comp
-L XR68C681:XR68C681CJTR-F IC1
+L mc68681-basic-rescue:XR68C681CJTR-F-XR68C681 IC1
 U 1 1 603DDDD7
 P 3400 3100
